Commit message: GICP working

File: src/surface_reconstruction/urdf/surface_reconstruction.urdf (robot description, URDF)
Before this commit: robot surface_reconstruction, 10 links, 9 joints
Links:
- added link laser_frame; visual box size=0.05 0.05 0.04
Joints:
- added joint dobot_to_laser: type fixed, parent Link6, child laser_frame, origin xyz=0 0 0.05 rpy=3.1415927 0 2.0944

Commit message: nav2 working sort of

File: src/surface_reconstruction/urdf/surface_reconstruction.urdf (robot description, URDF)
Before this commit: robot surface_reconstruction, 11 links, 10 joints
Joints:
- joint dobot_to_rslidar: origin xyz=0 0 0.05 rpy=0 0 -1.0472 -> xyz=0 0 0.05 rpy=0 0 1.0472

Commit message: final push

File: src/surface_reconstruction/urdf/surface_reconstruction.urdf (robot description, URDF)
Before this commit: robot surface_reconstruction, 11 links, 10 joints
Joints:
- joint ranger_to_dobot: origin xyz=-0.4 0 0.2 rpy=0 0 0 -> xyz=0.4 0 0.2 rpy=0 0 3.1415927
